Commit message: robot visualization

File: urdf_tutorial/urdf/03-origins.urdf (robot description, URDF)
Before this commit: robot origins, 2 links, 1 joints
Links:
- added link left_leg; visual box size=0.6 0.1 0.2
Joints:
- added joint base_to_left_leg: type fixed, parent base_link, child left_leg, origin xyz=0 0.22 -0.25
- joint base_to_right_leg: origin xyz=0 -0.22 0.25 -> xyz=0 -0.22 -0.25

File: urdf_tutorial/urdf/06-flexible.urdf (robot description, URDF)
Before this commit: robot visual, 16 links, 15 joints
Joints:
- joint gripper_extension: origin xyz=0.19 0 0.2 rpy=0 0 0 -> xyz=0.19 0 0.2 rpy=0 1.5 0
