Commit message: made it prettier

File: urdf_tutorial/urdf/dobot.urdf (robot description, URDF)
Before this commit: robot dobot, 10 links, 9 joints
Joints:
- joint joint_four: limit lower=0 upper=-1.5 effort=1000.0 velocity=0.5 -> lower=-0.3 upper=-1.7 effort=1000.0 velocity=0.5; origin xyz=0 0 ${link3_length+0.025} rpy=0 0 0 -> xyz=0 0 ${link3_length} rpy=0 0 0
- joint joint_three: limit lower=0 upper=-1.74 effort=1000.0 velocity=0.5 -> lower=-0.654 upper=-2.413 effort=1000.0 velocity=0.5
- joint joint_two: origin xyz=0 0 ${link1_heigth-0.01} rpy=0 0 0 -> xyz=0 0 ${link1_heigth} rpy=0 0 0

File: urdf_tutorial/urdf/dobot.urdf.xacro (robot description, xacro)
@@ -50,5 +50,5 @@
   <link name="link_1">
     <visual>
-     <origin xyz="0 0 ${link0_heigth}" rpy="0 0 0"/>
+     <origin xyz="0 0 ${link1_heigth/2}" rpy="0 0 0"/>
      <geometry>
       <box size="${link1_width} ${link1_width} ${link1_heigth}"/>
@@ -66,5 +66,5 @@
   <link name="link_2">
    <visual>
-    <origin xyz="0 0 ${link1_heigth}" rpy="0 0 0"/>
+    <origin xyz="0 0 ${link2_length/2}" rpy="0 0 0"/>
     <geometry>
      <cylinder length="${link2_length}" radius="${link2_width/2}"/>
@@ -82,5 +82,5 @@
   <link name="link_3">
    <visual>
-    <origin xyz="0 0 ${link1_heigth}" rpy="0 0 0"/>
+    <origin xyz="0 0 ${link3_length/2}" rpy="0 0 0"/>
     <geometry>
      <cylinder length="${link3_length}" radius="${link3_width/2}"/>
@@ -98,5 +98,5 @@
   <link name="link_4">
    <visual>
-    <origin xyz="0 0 ${link0_heigth/2}" rpy="0 0 0"/>
+    <origin xyz="0 0 ${link4_length/2-0.025}" rpy="0 0 0"/>
     <geometry>
      <cylinder length="${link4_length}" radius="${link4_width/2}"/>
@@ -112,5 +112,5 @@
   <link name="link_5">
    <visual>
-    <origin xyz="0 0 ${link4_length}" rpy="0 0 0"/>
+    <origin xyz="0 0 0" rpy="0 0 0"/>
     <geometry>
      <cylinder length="0" radius="0"/>
